Commit message: Added proof of concept for service creating an obstacle.

File: ProjetSupaero2017/catkin_ws/src/intel_teleop/intel_teleop_ground/Objects/cylinder.xacro (robot description, xacro)
@@ -48,4 +48,5 @@
   <gazebo reference="my_cylinder">
     <static>true</static>
+    <turnGravityOff>true</turnGravityOff>
     <material>Gazebo/Blue</material>
   </gazebo>

File: ProjetSupaero2017/catkin_ws/src/intel_teleop/intel_teleop_ground/object.urdf (robot description, URDF)
Before this commit: robot cylinder, 1 links, 0 joints
Links:
- link my_cylinder: geometry collision cylinder length=5 radius=1; visual cylinder length=5 radius=1

Commit message: Added proof of concept for service creating an obstacle.

File: ProjetSupaero2017/catkin_ws/src/intel_teleop/intel_teleop_ground/Objects/cylinder.xacro (robot description, xacro)
@@ -13,6 +13,6 @@
 <xacro:arg name="roll" default="0" />
 <xacro:property name="roll" value="$(arg roll)" />
-<xacro:arg name="pitch" default="0" />
-<xacro:property name="pitch" value="$(arg pitch)" />
+<xacro:arg name="yaw" default="0" />
+<xacro:property name="yaw" value="$(arg yaw)" />
 <xacro:arg name="radius" default="1" />
 <xacro:property name="radius" value="$(arg radius)" />
@@ -21,6 +21,6 @@
 <!-- Macro to place the box -->
 <!-- ^ means: use the value of the variable with the same name already defined -->
-<xacro:macro name="Origin" params="x:=^ y:=^ z:=^ roll:=^ pitch:=^">
-  <origin xyz="${x} ${y} ${z}" rpy="${DegToRad * roll} ${DegToRad * pitch} 0" />
+<xacro:macro name="Origin" params="x:=^ y:=^ z:=^ roll:=^ yaw:=^">
+  <origin xyz="${x} ${y} ${z}" rpy="${roll} 0 ${yaw}" />
 </xacro:macro>
 <!-- Macro to create the box -->
@@ -34,6 +34,6 @@
     <inertial>
       <xacro:Origin/>
-      <mass value="1.0" />
-      <inertia  ixx="0.0" ixy="0.0"  ixz="0.0"  iyy="0.0"  iyz="0.0"  izz="0.0" />
+      <mass value="1e9" />
+      <inertia  ixx="1e9" ixy="1e9"  ixz="1e9"  iyy="1e9"  iyz="1e9"  izz="1e9" />
     </inertial>
     <visual>
