Commit message: Updated node display -- launch file to display obstacles

File: ProjetSupaero2018/catkin_ws/src/display/urdf/cylinder.urdf (robot description, URDF)
Before this commit: robot cylinder, 1 links, 0 joints
Links:
- link my_cylinder: geometry collision cylinder length=1 radius=0.2; visual cylinder length=1 radius=0.2
