Commit message: nouvelle structure de fichier, récupération des fichiers obstacles.

File: ProjetSupaero2018/catkin_ws/src/display/models/cylinder/cylinder.urdf (robot description, URDF)
Before this commit: robot cylinder, 1 links, 0 joints
Links:
- link my_cylinder: geometry collision cylinder length=1 radius=0.4; visual cylinder length=1 radius=0.4

Commit message: Jalon 2 integrated but not working properly

File: ProjetSupaero2018/catkin_ws/src/display/models/cylinder/cylinder.urdf (robot description, URDF)
Before this commit: robot cylinder, 1 links, 0 joints
Links:
- link my_cylinder: geometry collision cylinder length=1 radius=1.0; visual cylinder length=1 radius=1.0

Commit message: Solved i+j -> N*i+j bug + traj client with many examples

File: ProjetSupaero2018/catkin_ws/src/display/models/cylinder/cylinder.urdf (robot description, URDF)
Before this commit: robot cylinder, 1 links, 0 joints
Links:
- link my_cylinder: geometry collision cylinder length=1 radius=2.0; visual cylinder length=1 radius=2.0
